File: mps-io.kicad_sch (KiCad schematic)
At the start: 56 parts, among them J1 PMOD, J2 430451628, U1 SN74AC16PWR, U2 TLP2312, U3 TLP2312, U4 TLP2312, U5 TLP2312, U6 ILQ615-4X009T, U7 SN74AC14PWR

Commit message: add missing symbols to 0local
Parts:
- J2: symbol 430451628:430451628 -> 0local:430451628
- U1: symbol SN74AC16PWR:SN74AC16PWR -> 0local:SN74AC16PWR
- U7: symbol SN74AC14PWR:SN74AC14PWR -> 0local:SN74AC14PWR

Commit message: update all symbols from libraries
Parts:
- D1: footprint 0local:LED_0603_1608Metric -> LED_SMD:LED_1206_3216Metric
- U2, U3, U4, U5: footprint 0local:SO6_TLP2312(V4-TPL,E -> SO6_TLP2312(V4-TPL,E
- U6: footprint 0local:ILQ615-4X009T_SMD-16 -> ILQ615-4X009T:SOIC254P1005X380-16N; MANUFACTURER (none) -> Vishay
Connections:
- net +3.3V: no longer TP1.1
- net GND: no longer TP2.1
Other:
- moved on the sheet: TP1, TP2
