File: mps-io.kicad_sch (KiCad schematic)
At the start: 56 parts, among them J1 PMOD, J2 430451628, U1 SN74AC16PWR, U2 TLP2312, U3 TLP2312, U4 TLP2312, U5 TLP2312, U6 ILQ615-4X009T, U7 SN74AC14PWR

Commit message: fixup footprint assignment
Parts:
- U2, U3, U4, U5: footprint SO6_TLP2312(V4-TPL,E -> 0local:SO6_TLP2312(V4-TPL,E
- U6: footprint ILQ615-4X009T:SOIC254P1005X380-16N -> 0local:ILQ615-4X009T_SMD-16
