File: mps-io.kicad_pcb (KiCad board)
At the start: 4 copper layers, 50 x 30 mm, 56 parts, among them J1 PMOD, J2 430451628, U1 SN74AC16PWR, U2 TLP2312, U3 TLP2312, U4 TLP2312, U5 TLP2312, U6 ILQ615-4X009T, U7 SN74AC14PWR

Commit message: fixup footprint assignment
Parts:
- D1: footprint 0local:LED_0603_1608Metric -> LED_SMD:LED_1206_3216Metric
