File: mps-io.kicad_pcb (KiCad board)
At the start: 4 copper layers, 50 x 30 mm, 56 parts, among them J1 PMOD, J2 430451628, U1 SN74AC16PWR, U2 TLP2312, U3 TLP2312, U4 TLP2312, U5 TLP2312, U6 ILQ615-4X009T, U7 SN74AC14PWR

Commit message: Add KiBot automation
Other:
- board text added: "0"
- board text added: "0 mm"
- board text added: "0.01 mm"
- board text added: "0.02"
- board text added: "0.035 mm"
- board text added: "0.1 mm"
- board text added: "0.2000 mm / 0.2000 mm"
- board text added: "0.2540 mm"
- board text added: "1"
- board text added: "1.24 mm"
- board text added: "1.6000 mm"
- board text added: "3.3"
- board text added: "4"
- board text added: "4.5"
- board text added: "50.0000 mm x 30.0000 mm"
- board text added: "B.Cu"
- board text added: "B.Mask"
- board text added: "B.Paste"
- board text added: "B.Silkscreen"
- board text added: "BOARD CHARACTERISTICS"
- board text added: "Board Thickness:"
- board text added: "Board overall dimensions:"
- board text added: "Bottom Silk Screen"
- board text added: "Bottom Solder Mask"
- board text added: "Bottom Solder Paste"
- board text added: "Castellated pads:"
- board text added: "Color"
- board text added: "Copper Finish:"
- board text added: "Copper Layer Count:"
- board text added: "Dielectric"
- board text added: "Edge card connectors:"
- board text added: "Epsilon R"
- board text added: "F.Cu"
- board text added: "F.Mask"
- board text added: "F.Paste"
- board text added: "F.Silkscreen"
- board text added: "FR4"
- board text added: "Impedance Control:"
- board text added: "In1.Cu"
- board text added: "In2.Cu"
- board text added: "Layer Name"
- board text added: "Loss Tangent"
- board text added: "Material"
- board text added: "Min hole diameter:"
- board text added: "Min track/spacing:"
- board text added: "No"
- board text added: "None"
- board text added: "Not specified"
- board text added: "Plated Board Edge:"
- board text added: "Thickness (mm)"
- board text added: "Top Silk Screen"
- board text added: "Top Solder Mask"
- board text added: "Top Solder Paste"
- board text added: "Type"
- board text added: "copper"
- board text added: "core"
- board text added: "prepreg"

Commit message: Final tweaks: J2 pads, D1 603, no mask backoffs, table updates
Parts:
- D1: footprint LED_SMD:LED_1206_3216Metric -> 0local:LED_0603_1608Metric
Other:
- board text added: "0.4000 mm"
- board text added: "Green"
- board text added: "White"
- board text removed: "0.2540 mm"

Commit message: Changed slot, moved R5-R8, added/moved slik
Parts:
- moved R5 11.3 mm to (113.6, 82.4), turned to 180 degrees
- moved R6 9.03 mm to (113.6, 84.4), turned to 180 degrees
- moved R7 7.11 mm to (113.6, 86.4), turned to 180 degrees
- moved R8 5.96 mm to (113.6, 88.4), turned to 180 degrees
Routing:
- net /OUT1: track 28.0 -> 17.2 mm
- net /OUT2: track 30.0 -> 21.8 mm
- net /OUT3: track 22.8 -> 15.4 mm
- net /OUT4: track 34.5 -> 30.0 mm
- net +3.3V: track 50.7 -> 53.5 mm
- net /IN4: track 14.9 -> 15.4 mm
Other:
- board text added: "+"
- board text added: "-"
- board text added: "2"
- board text added: "3"
- board text added: "I1"
- board text added: "I2"
- board text added: "I3"
- board text added: "I4"
- board text added: "MPS-IO V1.0"
- board text added: "O1"
- board text added: "O2"
- board text added: "O3"
- board text added: "O4"
- board text added: "Osprey DCS 2024"
- board text removed: "MPS-IO V1.0 2024"
- board text removed: "Osprey DCS"
